File: amoeba-choc.kicad_pcb (KiCad board)
At the start: 2 copper layers, 19 x 18 mm, 14 parts, among them J1 Conn_01x01_Male, J2 Conn_01x01_Male, J3 Conn_01x01_Male, J4 Conn_01x01_Male, J5 Conn_01x01_Male, J6 Conn_01x01_Male, J7 Conn_01x01_Male, J8 Conn_01x01_Male, SW1 SW_DIP_x02

Commit message: Added 2u footprint and cleanedup traces
A  Giri-Kailh-Choc-Library.pretty/Kailh-PG1350-2u-stabilizer-refined.kicad_mod
M  amoeba-choc.kicad_pcb
M  amoeba-choc.kicad_prl
M  amoeba-choc.kicad_sch
A  socket-2u/.gitignore
A  socket-2u/fp-lib-table
A  socket-2u/socket-2u.kicad_pcb
A  socket-2u/socket-2u.kicad_prl
A  socket-2u/socket-2u.kicad_pro
A  socket-2u/socket-2u.kicad_sch
Parts:
- added H5: MountingHole, Giri-Kailh-Choc-Library:MountingHole_1.2mm_M1, F.Cu at (127.4, 76.5)
- added H7: MountingHole, Giri-Kailh-Choc-Library:MountingHole_1.2mm_M1, F.Cu at (110.7, 76.5)
Routing:
- net Net-(D1-Pad2): track 23.3 -> 21.5 mm
- net Net-(J3-Pad1): track 18.0 -> 17.1 mm
Changed lines of the file:
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@@
+    (pad "" np_thru_hole circle (at 0 0) (size 1.2 1.2) (drill 1.2) (layers F&B.Cu *.Mask))
+  )
+  (footprint "Giri-Kailh-Choc-Library:MountingHole_1.2mm_M1" (layer "F.Cu")
+    (at 127.39 76.5)
+    (descr "Mounting Hole 2.1mm, no annular")
+    (tags "mounting hole 2.1mm no annular")
+    (property "Sheetfile" "amoeba-choc.kicad_sch")
+    (property "Sheetname" "")
+    (attr exclude_from_pos_files)
+    (fp_text reference "H5" (at 0 -3.2) (layer "F.Fab")
+      (effects (font (size 1 1) (thickness 0.15)))
+    )
+    (fp_text value "MountingHole" (at 0 3.2) (layer "F.Fab")
+      (effects (font (size 1 1) (thickness 0.15)))
+    )
+    (fp_text user "${REFERENCE}" (at 0 0) (layer "F.Fab")
+      (effects (font (size 1 1) (thickness 0.15)))
+    )
+    (fp_circle (center 0 0) (end 1.1 0) (layer "Cmts.User") (width 0.15) (fill none))
+    (fp_circle (center 0 0) (end 1.35 0) (layer "F.CrtYd") (width 0.05) (fill none))
     (pad "" np_thru_hole circle (at 0 0) (size 1.2 1.2) (drill 1.2) (layers F&B.Cu *.Mask))
   )
@@
     (pad "1" thru_hole rect (at 0 0) (size 2.5 1) (drill 0.5) (layers *.Cu *.Mask)
       (net 4 "Net-(J2-Pad1)") (pinfunction "Pin_1") (pintype "passive"))
+  )
+  (footprint "Giri-Kailh-Choc-Library:MountingHole_1.2mm_M1" (layer "F.Cu")
+    (at 110.74 76.5)
+    (descr "Mounting Hole 2.1mm, no annular")
+    (tags "mounting hole 2.1mm no annular")
+    (property "Sheetfile" "amoeba-choc.kicad_sch")
+    (property "Sheetname" "")
+    (attr exclude_from_pos_files)
+    (fp_text reference "H7" (at 0 -3.2) (layer "F.Fab")
+      (effects (font (size 1 1) (thickness 0.15)))
+    )
+    (fp_text value "MountingHole" (at 0 3.2) (layer "F.Fab")
+      (effects (font (size 1 1) (thickness 0.15)))
+    )
+    (fp_text user "${REFERENCE}" (at 0 0) (layer "F.Fab")
+      (effects (font (size 1 1) (thickness 0.15)))
+    )
+    (fp_circle (center 0 0) (end 1.1 0) (layer "Cmts.User") (width 0.15) (fill none))
+    (fp_circle (center 0 0) (end 1.35 0) (layer "F.CrtYd") (width 0.05) (fill none))
+    (pad "" np_thru_hole circle (at 0 0) (size 1.2 1.2) (drill 1.2) (layers F&B.Cu *.Mask))
   )
   (footprint "Giri-Kailh-Choc-Library:TestPoint_THTPad_1.0x2.5mm_Drill0.5mm" (layer "F.Cu")
@@
     (effects (font (size 0.5 0.5) (thickness 0.1)) (justify mirror))
   )
-  (gr_text "Kailh Choc 1350 Hotswap" (at 118.98 78.94) (layer "B.SilkS")
+  (gr_text "Kailh Choc 1350 Hotswap" (at 118.98 78.74) (layer "B.SilkS")
     (effects (font (size 0.2 0.2) (thickness 0.05)) (justify mirror))
   )
@@
     (effects (font (size 0.2 0.2) (thickness 0.05)) (justify mirror))
   )
-  (segment (start 121.915 81.885) (end 121.85 81.82) (width 0.25) (layer "B.Cu") (net 1))
   (segment (start 121.915 81.885) (end 121.965 81.885) (width 0.25) (layer "B.Cu") (net 1))
   (segment (start 121.965 81.885) (end 125.15 78.7) (width 0.25) (layer "B.Cu") (net 1))
-  (segment (start 126.78 73.59) (end 124.986843 73.59) (width 0.25) (layer "B.Cu") (net 2))
   (segment (start 121.85 76.11) (end 124.32 73.64) (width 0.25) (layer "B.Cu") (net 2))
   (segment (start 126.73 73.64) (end 126.78 73.59) (width 0.25) (layer "B.Cu") (net 2))
@@
   (segment (start 113.39 83.58) (end 113.39 81.86) (width 0.25) (layer "B.Cu") (net 5))
   (segment (start 113.39 81.86) (end 111.215 79.685) (width 0.25) (layer "B.Cu") (net 5))
-  (segment (start 114.065 78.935) (end 114.2 78.8) (width 0.25) (layer "B.Cu") (net 5))
-  (segment (start 114.065 79.685) (end 114.065 78.935) (width 0.25) (layer "B.Cu") (net 5))
 )
