File: amoeba-choc.kicad_sch (KiCad schematic)
At the start: 14 parts, among them J1 Conn_01x01_Male, J2 Conn_01x01_Male, J3 Conn_01x01_Male, J4 Conn_01x01_Male, J5 Conn_01x01_Male, J6 Conn_01x01_Male, J7 Conn_01x01_Male, J8 Conn_01x01_Male, SW1 SW_DIP_x02

Commit message: Added 2u footprint and cleanedup traces
A  Giri-Kailh-Choc-Library.pretty/Kailh-PG1350-2u-stabilizer-refined.kicad_mod
M  amoeba-choc.kicad_pcb
M  amoeba-choc.kicad_prl
M  amoeba-choc.kicad_sch
A  socket-2u/.gitignore
A  socket-2u/fp-lib-table
A  socket-2u/socket-2u.kicad_pcb
A  socket-2u/socket-2u.kicad_prl
A  socket-2u/socket-2u.kicad_pro
A  socket-2u/socket-2u.kicad_sch
Parts:
- added H5, H7: MountingHole, Giri-Kailh-Choc-Library:MountingHole_1.2mm_M1, symbol Mechanical:MountingHole
Changed lines of the file:
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@@
     (stroke (width 0) (type default) (color 0 0 0 0))
+  )
+  (symbol (lib_id "Mechanical:MountingHole") (at 104.14 72.39 0) (unit 1)
+    (in_bom yes) (on_board yes) (fields_autoplaced)
+    (property "Reference" "H5" (id 0) (at 106.68 71.5553 0)
+      (effects (font (size 1.27 1.27)) (justify left))
+    )
+    (property "Value" "MountingHole" (id 1) (at 106.68 74.0922 0)
+      (effects (font (size 1.27 1.27)) (justify left))
+    )
+    (property "Footprint" "Giri-Kailh-Choc-Library:MountingHole_1.2mm_M1" (id 2) (at 104.14 72.39 0)
+      (effects (font (size 1.27 1.27)) hide)
+    )
+    (property "Datasheet" "~" (id 3) (at 104.14 72.39 0)
+      (effects (font (size 1.27 1.27)) hide)
+    )
   )
   (symbol (lib_id "Mechanical:MountingHole") (at 104.14 52.07 0) (unit 1)
@@
     )
   )
+  (symbol (lib_id "Mechanical:MountingHole") (at 104.14 87.63 0) (unit 1)
+    (in_bom yes) (on_board yes) (fields_autoplaced)
+    (property "Reference" "H7" (id 0) (at 106.68 86.7953 0)
+      (effects (font (size 1.27 1.27)) (justify left))
+    )
+    (property "Value" "MountingHole" (id 1) (at 106.68 89.3322 0)
+      (effects (font (size 1.27 1.27)) (justify left))
+    )
+    (property "Footprint" "Giri-Kailh-Choc-Library:MountingHole_1.2mm_M1" (id 2) (at 104.14 87.63 0)
+      (effects (font (size 1.27 1.27)) hide)
+    )
+    (property "Datasheet" "~" (id 3) (at 104.14 87.63 0)
+      (effects (font (size 1.27 1.27)) hide)
+    )
+  )
   (symbol (lib_id "Mechanical:MountingHole") (at 104.14 58.42 0) (unit 1)
     (in_bom yes) (on_board yes) (fields_autoplaced)
@@
       (reference "H4") (unit 1) (value "MountingHole") (footprint "Giri-Kailh-Choc-Library:MountingHole_1.2mm_M1")
     )
+    (path "/056c9c13-522f-449c-84bd-83c95f6465a1"
+      (reference "H5") (unit 1) (value "MountingHole") (footprint "Giri-Kailh-Choc-Library:MountingHole_1.2mm_M1")
+    )
+    (path "/80aa8240-b182-45b1-bd96-4b2cb6340d6c"
+      (reference "H7") (unit 1) (value "MountingHole") (footprint "Giri-Kailh-Choc-Library:MountingHole_1.2mm_M1")
+    )
     (path "/cb6e11c9-9471-4a9b-9af5-208d08897519"
